File: FPGA_board-v1.sch (EAGLE design)
At the start: 81 parts, among them IC1 7805T, IC15 74LS365D, IC16 74LS365D, IC17 74LS365D, IC18 74LS365D, IC19 74LS365D, IC2 7805T, IC20 74LS365D, IC21 74LS365D, IC22 74LS365D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

Commit message: Add files via upload
Parts:
- removed J10, J11, J12: (no value), SparkFun-Connectors:CONN_10"
Connections:
- net 5V_ESP: no longer J10.10
- net EN: now also S1.S@1
- net ESP_RX: now also S2.S@1; no longer J11.2
- net ESP_TX: now also S3.S@1; no longer J11.3
- net GND: now also S1.P, S2.P, S3.P; no longer J10.8
Changed lines of the file:
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@@
 <part name="C9" library="rcl" deviceset="C-EU" device="C1206" value="47uF"/>
 <part name="C10" library="rcl" deviceset="C-EU" device="C1206" value="47uF"/>
-<part name="J10" library="SparkFun-Connectors" library_urn="urn:adsk.eagle:library:513" deviceset="CONN_10" device="&quot;" package3d_urn="urn:adsk.eagle:package:38157/1"/>
-<part name="J11" library="SparkFun-Connectors" library_urn="urn:adsk.eagle:library:513" deviceset="CONN_10" device="&quot;" package3d_urn="urn:adsk.eagle:package:38157/1"/>
-<part name="J12" library="SparkFun-Connectors" library_urn="urn:adsk.eagle:library:513" deviceset="CONN_10" device="&quot;" package3d_urn="urn:adsk.eagle:package:38157/1"/>
 </parts>
 <sheets>
@@
 <attribute name="VALUE" x="-766.496" y="-632.699" size="1.778" layer="96"/>
 </instance>
-<instance part="J10" gate="G$1" x="-556.26" y="-553.72" smashed="yes">
-<attribute name="VALUE" x="-556.26" y="-576.326" size="1.778" layer="96" font="vector"/>
-<attribute name="NAME" x="-556.26" y="-545.592" size="1.778" layer="95" font="vector"/>
-</instance>
-<instance part="J11" gate="G$1" x="-530.86" y="-553.72" smashed="yes">
-<attribute name="VALUE" x="-530.86" y="-576.326" size="1.778" layer="96" font="vector"/>
-<attribute name="NAME" x="-530.86" y="-545.592" size="1.778" layer="95" font="vector"/>
-</instance>
-<instance part="J12" gate="G$1" x="-510.54" y="-551.18" smashed="yes">
-<attribute name="VALUE" x="-510.54" y="-573.786" size="1.778" layer="96" font="vector"/>
-<attribute name="NAME" x="-510.54" y="-543.052" size="1.778" layer="95" font="vector"/>
-</instance>
 </instances>
 <busses>
@@
 </segment>
 <segment>
+<pinref part="S2" gate="1" pin="P@1"/>
+<pinref part="S2" gate="1" pin="P"/>
+<wire x1="-810.26" y1="-706.12" x2="-810.26" y2="-703.58" width="0.1524" layer="91"/>
+<label x="-815.34" y="-706.12" size="1.778" layer="95"/>
+</segment>
+<segment>
 <pinref part="S3" gate="1" pin="P@1"/>
+<pinref part="S3" gate="1" pin="P"/>
+<wire x1="-810.26" y1="-716.28" x2="-810.26" y2="-713.74" width="0.1524" layer="91"/>
 <label x="-815.34" y="-716.28" size="1.778" layer="95"/>
-<wire x1="-810.26" y1="-716.28" x2="-815.34" y2="-716.28" width="0.1524" layer="91"/>
 </segment>
 <segment>
@@
 </segment>
 <segment>
+<pinref part="S1" gate="1" pin="P"/>
+<pinref part="S1" gate="1" pin="P@1"/>
+<wire x1="-734.06" y1="-769.62" x2="-734.06" y2="-772.16" width="0.1524" layer="91"/>
+<wire x1="-734.06" y1="-769.62" x2="-736.6" y2="-769.62" width="0.1524" layer="91"/>
+<junction x="-734.06" y="-769.62"/>
+<label x="-739.14" y="-769.62" size="1.778" layer="95"/>
+</segment>
+<segment>
 <pinref part="JP1" gate="A" pin="19"/>
 <wire x1="-924.56" y1="-678.18" x2="-937.26" y2="-678.18" width="0.1524" layer="91"/>
@@
 <label x="-911.86" y="-678.18" size="1.778" layer="95"/>
 </segment>
-<segment>
-<pinref part="S1" gate="1" pin="P@1"/>
-<wire x1="-734.06" y1="-772.16" x2="-736.6" y2="-772.16" width="0.1524" layer="91"/>
-<label x="-741.68" y="-772.16" size="1.778" layer="95"/>
-</segment>
-<segment>
-<pinref part="S2" gate="1" pin="P@1"/>
-<wire x1="-810.26" y1="-706.12" x2="-812.8" y2="-706.12" width="0.1524" layer="91"/>
-<label x="-815.34" y="-706.12" size="1.778" layer="95"/>
-</segment>
-<segment>
-<pinref part="J10" gate="G$1" pin="8"/>
-<wire x1="-546.1" y1="-553.72" x2="-543.56" y2="-553.72" width="0.1524" layer="91"/>
-<label x="-543.56" y="-553.72" size="1.778" layer="95"/>
-</segment>
 </net>
 <net name="M21" class="6">
@@
 </segment>
 <segment>
+<pinref part="S2" gate="1" pin="S@1"/>
 <pinref part="S2" gate="1" pin="S"/>
-<label x="-800.1" y="-703.58" size="1.778" layer="95"/>
-<wire x1="-800.1" y1="-703.58" x2="-797.56" y2="-703.58" width="0.1524" layer="91"/>
-</segment>
-<segment>
-<pinref part="J11" gate="G$1" pin="2"/>
-<wire x1="-520.7" y1="-568.96" x2="-518.16" y2="-568.96" width="0.1524" layer="91"/>
-<label x="-520.7" y="-568.96" size="1.778" layer="95"/>
+<wire x1="-800.1" y1="-706.12" x2="-800.1" y2="-703.58" width="0.1524" layer="91"/>
+<label x="-802.64" y="-706.12" size="1.778" layer="95"/>
 </segment>
 </net>
@@
 </segment>
 <segment>
+<pinref part="S3" gate="1" pin="S@1"/>
 <pinref part="S3" gate="1" pin="S"/>
-<label x="-800.1" y="-713.74" size="1.778" layer="95"/>
-<wire x1="-800.1" y1="-713.74" x2="-795.02" y2="-713.74" width="0.1524" layer="91"/>
+<wire x1="-800.1" y1="-716.28" x2="-800.1" y2="-713.74" width="0.1524" layer="91"/>
+<label x="-802.64" y="-713.74" size="1.778" layer="95"/>
 </segment>
 <segment>
@@
 <label x="-601.98" y="-728.98" size="1.778" layer="95" grouprefs="BUFFER"/>
 </segment>
-<segment>
-<pinref part="J11" gate="G$1" pin="3"/>
-<wire x1="-520.7" y1="-566.42" x2="-518.16" y2="-566.42" width="0.1524" layer="91"/>
-<label x="-520.7" y="-566.42" size="1.778" layer="95"/>
-</segment>
 </net>
 <net name="_ESP_EN" class="3">
@@
 <pinref part="S1" gate="1" pin="S"/>
 <pinref part="R8" gate="G$1" pin="1"/>
+<pinref part="S1" gate="1" pin="S@1"/>
+<wire x1="-723.9" y1="-772.16" x2="-723.9" y2="-769.62" width="0.1524" layer="91"/>
+<junction x="-723.9" y="-769.62"/>
+<label x="-723.9" y="-774.7" size="1.778" layer="95"/>
 </segment>
 </net>
@@
 <label x="-767.08" y="-622.3" size="1.778" layer="95"/>
 </segment>
-<segment>
-<pinref part="J10" gate="G$1" pin="10"/>
-<wire x1="-546.1" y1="-548.64" x2="-543.56" y2="-548.64" width="0.1524" layer="91"/>
-<label x="-543.56" y="-548.64" size="1.778" layer="95"/>
-</segment>
 </net>
