File: FPGA_board-v1.brd (EAGLE design)
At the start: 171.1 x 156.7 mm, 82 parts, among them IC1 7805T, IC15 74LS365D, IC16 74LS365D, IC17 74LS365D, IC18 74LS365D, IC19 74LS365D, IC2 7805T, IC20 74LS365D, IC21 74LS365D, IC22 74LS365D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

Commit message: Added latest versions of main board
Parts:
- removed J10, J11, J12: (no value), SparkFun-Connectors:1X10
- moved S3 4.03 mm to (-18.7, -53.9)
- moved S2 3.45 mm to (-18.8, -42.3)
Connections:
- net 5V_ESP: no longer J10.10
- net EN: now also S1.5
- net ESP_RX: now also S2.5; no longer J11.2
- net ESP_TX: now also S3.5; no longer J11.3
- net GND: now also S1.2, S2.2, S3.2; no longer J10.8
Routing:
- net EN: track 453.0 -> 461.7 mm
- net ESP_RX: track 53.9 -> 60.2 mm
- net ESP_TX: track 61.5 -> 67.2 mm
